Commit message: 2nd commit -- pick and place problem

File: cobot_simulation/urdf/gripper.xacro (robot description, xacro)
@@ -1,4 +1,5 @@
 <?xml version = "1.0"?>
 <robot name="cobot" xmlns:xacro="http://www.ros.org/wiki/xacro">
+    <xacro:include filename="$(find cobot_simulation)/urdf/joint_link.xacro"/>
     <!-- Model a gripper -->
     <xacro:macro name="gripper" params="parent origin_xyz">
@@ -11,5 +12,5 @@
             <axis xyz="0 0 1"/>
             <limit lower="-3.14" upper="3.14" velocity="0.5" effort="200"/>
-            <origin xyz="{origin_xyz}" rpy="0 0 0"/>
+            <origin xyz="${origin_xyz}" rpy="0 0 0"/>
             <dynamics damping="1" friction="1"/>
         </joint>
@@ -24,7 +25,7 @@
             <limit lower="0" upper="0.055" velocity="0.5" effort="200"/>
             <origin xyz="0 -0.065 0.03" rpy="0 0 0"/>
-            <dynamics damping="1" friction="1"/>
+            <dynamics damping="1" friction="2"/>
         </joint>
-        <xacro:transmission name="trans_gripper_right_joint" joint_name="gripper_right" actuator_name="motor_gripper_right_joint"/>
+        <xacro:transmission name="trans_gripper_right_joint" joint_name="gripper_right_joint" actuator_name="motor_gripper_right_joint"/>
         <!-- Gripper left -->
         <xacro:cobot_link_box name="gripper_left" origin_xyz="0.0 0.0 0.05" origin_rpy="0 0 0" size="0.01 0.01 0.1" mass="0.5"
@@ -36,12 +37,12 @@
             <limit lower="-0.055" upper="0" velocity="0.5" effort="200"/>
             <origin xyz="0 0.065 0.03" rpy="0 0 0"/>
-            <dynamics damping="1" friction="1"/>
+            <dynamics damping="1" friction="2"/>
             <mimic joint="gripper_right_joint" multiplier="-1.0" offset="0"/>
         </joint>
-        <xacro:transmission name="trans_gripper_left_joint" joint_name="gripper_left" actuator_name="motor_gripper_left_joint"/>
+        <xacro:transmission name="trans_gripper_left_joint" joint_name="gripper_left_joint" actuator_name="motor_gripper_left_joint"/>
         <!-- ros control plugin with mimic-->
         <xacro:macro name="mimic_joint_plugin_gazebo" params="parent_joint mimic_joint has_pid:=false multiplier:=-1.0 offset:=0 sensitiveness:=0.0 max_effort:=200 robot_namespace:='/cobot'">
             <gazebo>
-                <plugin name="${mimic_joint}_mimic_joint_plugin" filename="libroboticsgroup_gazebo_mimic_joint_plugin.so">
+                <plugin name="${mimic_joint}_mimic_joint_plugin" filename="libroboticsgroup_upatras_gazebo_mimic_joint_plugin.so">
                     <joint>${parent_joint}</joint>
                     <mimicJoint>${mimic_joint}</mimicJoint>

File: cobot_simulation/urdf/joint_link.xacro (robot description, xacro)
@@ -56,8 +56,8 @@
             <type>transmission_interface/SimpleTransmission</type>
             <joint name="${joint_name}">
-                <hardwareInterface>hardware_interface/EffortJointInterface</hardwareInterface>
+                <hardwareInterface>hardware_interface/PositionJointInterface</hardwareInterface>
             </joint>
             <actuator name="${actuator_name}">
-                <hardwareInterface>hardware_interface/EffortJointInterface</hardwareInterface>
+                <hardwareInterface>hardware_interface/PositionJointInterface</hardwareInterface>
                 <mechanicalReduction>1</mechanicalReduction>
             </actuator>
